File: portal/portal-hw/portal.brd (EAGLE design)
At the start: 137 x 61 mm, 43 parts, among them IC1 RT9742GGJ5, IC4 TPD4EUSB30DQAR, IC5 AP64501SP-13, J1 CON-SD-CARD_MICROSD-2908-05, J2 615008137421, J4 61400416021, J5 629105150521, J6 POWER_JACKSLT, U1 FSUSB42MUX

Commit message: pcb work
Parts:
- removed J5: 629105150521, Wurth_Connectors_WR-USB:629105150521
- added C11, C12, C13, C14, C16, C17, C18, C19, C20, C22: 10u, rcl:C0805
- added C15, C21: 100u, Capacitor:CAPMP7343X310N
- added C23: 10u 30v, Capacitor:CAPMP7343X310N
- added IC6, IC7: AP22653W6-7, AP22653W6-7:SOT95P280X145-6N
- added J7: 614105150721, Wurth_Connectors_WR-USB:614105150721
- added R11, R12: 36k, rcl:R0805
- C3: value 10n 30v -> 10u 30v; device rcl:C0805 -> Capacitor:CAPMP7343X310N
- moved C10 377.8 mm to (158.0, 30.0)
- moved C9 367.0 mm to (157.0, 23.0)
- moved C8 358.5 mm to (152.0, 23.0)
- moved R10 351.5 mm to (123.8, 46.0), turned to 180 degrees
- moved R9 343.4 mm to (119.6, 46.0), turned to 180 degrees
- moved C7 339.7 mm to (119.6, 48.2)
- moved L1 317.8 mm to (117.0, 34.7), turned to 270 degrees
- moved C5 315.7 mm to (119.6, 41.8)
- moved C4 312.6 mm to (126.0, 38.0), turned to 180 degrees
- moved C2 308.0 mm to (128.2, 46.0), turned to 180 degrees
- moved C3 305.2 mm to (128.0, 32.0)
- moved R8 303.8 mm to (119.6, 43.9)
- moved C6 302.5 mm to (97.0, 37.4)
- moved IC5 296.7 mm to (126.0, 42.0), turned to 180 degrees
- moved IC4 204.2 mm to (-82.0, 52.0)
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Connections:
- removed net +5VPOWER: J3.18
- new net HDMI_5V: C17.1, C18.1, C19.1, C20.1, C21.1, IC7.6, J3.18
- new net N$4: IC6.5, R11.2
- new net VBUS: C11.1, C12.1, C13.1, C14.1, C15.1, IC6.6, J4.1
- new net VBUS_OTG: IC6.3, J7.1, R6.1, R7.2
- net +5V: now also C16.1, C22.1, C3.1, IC6.1, IC7.1, IC7.3; no longer J4.1
- net GND: now also C11.2, C12.2, C13.2, C14.2, C15.2, C16.2, C17.2, C18.2, C19.2, C20.2, C21.2, C22.2, C23.2, IC6.2, IC7.2, J7.5, J7.S1, J7.S2, R11.1, R12.1; no longer J5.5, J5.S1, J5.S2, J5.S3, J5.S4
- net N$11: now also J7.3; no longer J5.3
- net N$13: now also J7.2; no longer J5.2
- net N$18: now also IC7.5, R12.2; no longer J5.1, R6.1, R7.2
- net N$30: now also C23.1; no longer C3.1
Routing:
- net N$6: track 0.00 -> 14.1 mm
- net SD_PWR: track 0.00 -> 14.0 mm
- net N$33: track 0.00 -> 10.1 mm
- net N$36: track 0.00 -> 6.78 mm
- net N$30: track 0.00 -> 5.88 mm
- net N$31: track 0.00 -> 3.41 mm
- net N$34: track 0.00 -> 3.32 mm
- net N$32: track 0.00 -> 2.28 mm
- net N$35: track 0.00 -> 2.10 mm
