File: portal/portal-hw/portal.sch (EAGLE design)
At the start: 43 parts, among them IC1 RT9742GGJ5, IC4 TPD4EUSB30DQAR, IC5 AP64501SP-13, J1 CON-SD-CARD_MICROSD-2908-05, J2 615008137421, J4 61400416021, J5 629105150521, J6 POWER_JACKSLT, U1 FSUSB42MUX

Commit message: pcb work
Parts:
- removed J5: 629105150521, Wurth_Connectors_WR-USB:629105150521
- added C11, C12, C13, C14, C16, C17, C18, C19, C20, C22: 10u, rcl:C-EUC0805
- added C15, C21: 100u, Capacitor:C-POL_TANTALUM-2917(7343-METRIC)
- added C23: 10u 30v, Capacitor:C-POL_TANTALUM-2917(7343-METRIC)
- added IC6, IC7: AP22653W6-7, AP22653W6-7:AP22653W6-7
- added J7: 614105150721, Wurth_Connectors_WR-USB:614105150721
- added R11, R12: 36k, rcl:R-EU_R0805
- C3: value 10n 30v -> 10u 30v; device rcl:C-EUC0805 -> Capacitor:C-POL_TANTALUM-2917(7343-METRIC)
Connections:
- new net HDMI_5V: C17.1, C18.1, C19.1, C20.1, C21.+, IC7.OUT, J3.+5VPOWER
- new net N$4: IC6.ILIM, R11.2
- new net VBUS: C11.1, C12.1, C13.1, C14.1, C15.+, IC6.OUT, J4.VBUS
- new net VBUS_OTG: IC6.EN/!EN, J7.VBUS, R6.1, R7.2
- net +5V: now also C16.1, C22.1, C3.+, IC6.IN, IC7.EN/!EN, IC7.IN; no longer J4.VBUS
- net GND: now also C11.2, C12.2, C13.2, C14.2, C15.-, C16.2, C17.2, C18.2, C19.2, C20.2, C21.-, C22.2, C23.-, C3.-, IC6.GND, IC7.GND, J7.GND, J7.SHIELD, R11.1, R12.1; no longer C3.2, J5.GND, J5.SHIELD
- net N$11: now also J7.D+; no longer J5.D+
- net N$13: now also J7.D-; no longer J5.D-
- net N$18: now also IC7.ILIM, R12.2; no longer J5.VBUS, R6.1, R7.2
- net N$30: now also C23.+; no longer C3.1
Other:
- note added: "Todo: HDMI +5v Vertical Internal Micro USB"
- note removed: "Todo: HDMI +5v USB Power limit Vertical Internal Micro USB"
